File: pcb/keyboard/thingy.kicad_pcb (KiCad board)
At the start: 2 copper layers, 226.7 x 54 mm, 47 parts, among them J1 Conn_02x09_Odd_Even, J10 Conn_01x04_Socket, J11 Conn_01x06_Pin, J12 Conn_01x06_Pin, J14 Conn_01x04_Socket, J16 Conn_01x04_MountingPin, J2 Conn_01x02_Socket, J3 Conn_01x02_Socket, J4 Conn_01x02_Socket, J5 Raspberry_Pi_2_3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

Commit message: tidy up keyboard
tidy up keyboard schematic and break out pi serial interfaces
Parts:
- removed J6: Conn_01x07_Socket, Connector_PinSocket_2.54mm:PinSocket_1x07_P2.54mm_Vertical
- added J13: Conn_01x06, Connector_JST:JST_SH_BM06B-SRSS-TB_1x06-1MP_P1.00mm_Vertical, B.Cu at (-77.0, -3.80)
- added J15: Conn_01x06, Connector_JST:JST_SH_BM06B-SRSS-TB_1x06-1MP_P1.00mm_Vertical, B.Cu at (-77.0, 0.50)
- added J17: Conn_01x06, Connector_JST:JST_SH_BM06B-SRSS-TB_1x06-1MP_P1.00mm_Vertical, B.Cu at (-68.4, 0.50)
- added J18: Conn_01x06, Connector_JST:JST_SH_BM06B-SRSS-TB_1x06-1MP_P1.00mm_Vertical, B.Cu at (-59.8, -3.80)
- added J19: Conn_01x06, Connector_JST:JST_SH_BM06B-SRSS-TB_1x06-1MP_P1.00mm_Vertical, B.Cu at (-59.8, 0.50)
- moved J7 31.9 mm to (-76.6, 9.70), turned to -90 degrees
- moved J16 30.7 mm to (-68.4, -4.10)
- moved J9 4.49 mm to (-41.0, 0.00)
- moved J10 0.80 mm to (-18.4, -6.10)
Connections:
- net Net-(D1-DIN) renamed /SPI3_CS
- J16 pad 1: /SCL_P -> /I2C2_SCL
- J16 pad 2: /SDA_P -> /I2C2_SDA
- J5 pad 11: unconnected-(J5-GPIO17-Pad11) -> /SPI1_CS1
- J5 pad 12: unconnected-(J5-GPIO18/PWM0-Pad12) -> /SPI1_CS0
- J5 pad 13: unconnected-(J5-GPIO27-Pad13) -> /SDIO_D3
- J5 pad 15: unconnected-(J5-GPIO22-Pad15) -> /SDIO_CLK
- J5 pad 16: unconnected-(J5-GPIO23-Pad16) -> /SDIO_CMD
- J5 pad 17: unconnected-(J5-3V3-Pad17) -> +3.3VP
- J5 pad 18: unconnected-(J5-GPIO24-Pad18) -> /SDIO_D0
- J5 pad 19: /MOSI -> /UART3_CTS
- J5 pad 21: /MISO -> /UART3_RX
- J5 pad 22: unconnected-(J5-GPIO25-Pad22) -> /SDIO_D1
- J5 pad 23: /SCLK -> /UART3_RTS
- J5 pad 24: /CS -> /UART3_TX
- J5 pad 26: unconnected-(J5-~{CE1}/GPIO7-Pad26) -> /SPI3_SCLK
- J5 pad 27: unconnected-(J5-ID_SD/GPIO0-Pad27) -> /UART1_TX
- J5 pad 28: unconnected-(J5-ID_SC/GPIO1-Pad28) -> /UART1_RX
- J5 pad 29: unconnected-(J5-GCLK1/GPIO5-Pad29) -> /SPI3_MISO
- J5 pad 3: /SDA_P -> /UART1_CTS
- J5 pad 31: unconnected-(J5-GCLK2/GPIO6-Pad31) -> /SPI3_MOSI
- J5 pad 32: unconnected-(J5-PWM0/GPIO12-Pad32) -> /I2C2_SDA
- J5 pad 33: unconnected-(J5-PWM1/GPIO13-Pad33) -> /I2C2_SCL
- J5 pad 35: unconnected-(J5-GPIO19/MISO1-Pad35) -> /SPI1_MISO
- J5 pad 37: unconnected-(J5-GPIO26-Pad37) -> /SDIO_D2
- J5 pad 38: unconnected-(J5-GPIO20/MOSI1-Pad38) -> /SPI1_MOSI
- J5 pad 40: unconnected-(J5-GPIO21/SCLK1-Pad40) -> /SPI1_SCLK
- J5 pad 5: /SCL_P -> /UART1_RTS
- J7 pad 1: +5P -> unconnected-(J7-Pin_1-Pad1)
- J7 pad 3: Net-(J7-Pin_3) -> +3.3VP
- J7 pad 4: /MOSI -> /SPI3_MOSI
- J7 pad 5: /MISO -> /SPI3_MISO
- J7 pad 6: /SCLK -> /SPI3_SCLK
- J7 pad 7: Net-(J7-Pin_7) -> unconnected-(J7-Pin_7-Pad7)
Routing:
- net +3.3VP: track 10.1 -> 66.6 mm, vias 1 -> 0
- net /SPI1_CS1: track 0.00 -> 37.1 mm, vias 0 -> 1
- net /SPI3_CS: track 11.5 -> 48.3 mm, vias 0 -> 1
- net /SPI1_CS0: track 0.00 -> 35.4 mm, vias 0 -> 1
- net /UART1_CTS: track 0.00 -> 34.0 mm, vias 0 -> 1
- net /UART1_RTS: track 0.00 -> 27.7 mm, vias 0 -> 1
- net +5P: track 25.3 -> 4.12 mm
- net /SPI3_SCLK: track 0.00 -> 13.8 mm
- net /I2C2_SCL: track 0.00 -> 13.8 mm, vias 0 -> 1
- net /MOSI: track 13.4 -> 0.00 mm
- net /SCLK: track 13.4 -> 0.00 mm
- net /MISO: track 13.4 -> 0.00 mm
- net /UART3_CTS: track 0.00 -> 12.5 mm, vias 0 -> 1
- net /SPI3_MISO: track 0.00 -> 12.1 mm
- net /UART1_TX: track 0.00 -> 12.1 mm, vias 0 -> 1
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- added copper zone on In2.Cu, net +BATT
- added copper zone on In1.Cu, net -BATT
- added copper zone on In2.Cu, net -BATT
- added copper zone on In1.Cu, net GND
- added copper zone on In2.Cu, net GND
Other:
- outline, holes or cut-outs redrawn
- copper layers 2 -> 4
- board text removed: "USE ONLY SEEEDUINO XIAO ESP32-C6/S3"
